File: schematics_and_pcbs/imac_g3_333mhz_slot_loading_J20_adapter_board/imac_g3_333mhz_slot_loading_J20_adapter_board.kicad_pcb (KiCad board)
At the start: 2 copper layers, 82.6 x 51.7 mm, 12 parts, among them J1 DB15_Female_HighDensity, J20 Conn_02x10_Odd_Even, U1 ATmega328-PU, U2 ATmega328-PU, Y1 Crystal, Y2 Crystal

Commit message: made board a little curvier
Parts:
- C1, C2, C3, C4, Y1, Y2: moved to B.Cu
- moved U1 16.6 mm to (194.5, 65.3), turned to 0 degrees
- moved Y2 13.8 mm to (162.3, 82.8)
- moved C1 11.9 mm to (206.4, 89.7)
- moved C4 11.5 mm to (142.7, 84.0)
- moved Y1 11.3 mm to (188.7, 83.5), turned to 180 degrees
- moved U2 10.3 mm to (147.4, 65.4), turned to 0 degrees
- moved C2 8.85 mm to (212.9, 79.7)
- moved C3 7.33 mm to (136.8, 94.0)
- moved J20 6.11 mm to (189.1, 68.1)
Other:
- board size 82.6 x 51.7 mm -> 82.6 x 45.9 mm

Commit message: made more changes to the board
Parts:
- removed H2: MountingHole, MountingHole:MountingHole_3.5mm_Pad
- added D1: D_Schottky_ALT, Diode_THT:D_DO-41_SOD81_P7.62mm_Horizontal, B.Cu at (183.5, 86.1)
- added D2: D_Schottky_ALT, Diode_THT:D_DO-41_SOD81_P7.62mm_Horizontal, F.Cu at (172.1, 83.6)
- added J2: Screw_Terminal_01x06, TerminalBlock_Phoenix:TerminalBlock_Phoenix_PT-1,5-6-5.0-H_1x06_P5.00mm_Horizontal, F.Cu at (141.6, 72.1)
- added R1: 220, Resistor_THT:R_Axial_DIN0207_L6.3mm_D2.5mm_P7.62mm_Horizontal, B.Cu at (172.7, 75.3)
- added R2: 10k, Resistor_THT:R_Axial_DIN0207_L6.3mm_D2.5mm_P7.62mm_Horizontal, B.Cu at (205.2, 93.0)
- added U3: LCC110, Package_DIP:DIP-8_W7.62mm, F.Cu at (184.2, 75.3)
- H1: value MountingHole -> MountingHole_Pad
- Y1, Y2: moved to F.Cu
- moved C4 28.4 mm to (170.8, 79.8), turned to 0 degrees
- moved C3 27.0 mm to (162.6, 86.1)
- moved Y1 23.5 mm to (210.2, 93.1), turned to 270 degrees
- moved Y2 5.93 mm to (166.4, 78.5), turned to 270 degrees
- moved C2 2.48 mm to (212.7, 77.2)
- moved C1 2.35 mm to (206.4, 87.4)
- moved U2 1.84 mm to (149.2, 65.4)
Connections:
- H1 pad 1: (no net) -> GND
- J1 pad 6: /GND_RED -> GND
- J1 pad 7: /GND_GREEN -> GND
- J1 pad 8: /GND_BLUE -> GND
- J20 pad 10: /PFW -> /LPIACT:L1_LP
- J20 pad 14: /GND_BLUE -> GND
- J20 pad 16: /GND_GREEN -> GND
- J20 pad 18: /GND_RED -> GND
- U1 pad 19: Net-(U1-Pad19) -> /PWR_BTN
- U2 pad 20: /COMPUTER_5V -> Net-(D1-Pad1)
- U2 pad 7: /COMPUTER_5V -> Net-(D1-Pad1)
Routing:
- net GND: track 0.00 -> 262.0 mm
- net /PWR_BTN: track 0.00 -> 92.4 mm
- net /LPIACT:L1_LP: track 0.00 -> 82.3 mm
- net /COMPUTER_SDA: track 0.00 -> 70.0 mm
- net /DCO: track 0.00 -> 68.3 mm
- net /5V_TRICKLE: track 0.00 -> 57.2 mm
- net /PROT: track 0.00 -> 48.0 mm
- net /-10V: track 0.00 -> 47.4 mm
- net Net-(C2-Pad1): track 0.00 -> 40.9 mm
- net Net-(D1-Pad1): track 0.00 -> 40.4 mm
- net /COMPUTER_SCL: track 0.00 -> 38.5 mm, vias 0 -> 1
- net /V_SYNC: track 0.00 -> 37.6 mm, vias 0 -> 1
- net /H_SYNC: track 0.00 -> 36.9 mm
- net Net-(C1-Pad2): track 0.00 -> 31.6 mm
- net /LINE_SENSE: track 0.00 -> 28.9 mm
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- added copper zone on B.Cu, net GND
- added copper zone on F.Cu, net GND
Other:
- board text added: "PWR-BTN"
- board text added: "PWR/LED"
- board text added: "SNS"

Commit message: added caps to the board
Parts:
- added C5: 470uF, Capacitor_THT:CP_Radial_D8.0mm_P3.50mm, F.Cu at (208.3, 95.0)
- added C6: 470uF, Capacitor_THT:CP_Radial_D8.0mm_P3.50mm, F.Cu at (142.2, 105.2)
- added JP1: SolderJumper_2_Open, Jumper:SolderJumper-2_P1.3mm_Open_RoundedPad1.0x1.5mm, B.Cu at (176.3, 106.7)
- added JP2: SolderJumper_2_Open, Jumper:SolderJumper-2_P1.3mm_Open_RoundedPad1.0x1.5mm, B.Cu at (166.6, 106.7)
- C1, C2, C3, C4, D1, R1, R2: moved to F.Cu
- moved Y2 32.1 mm to (149.4, 105.7), turned to 0 degrees
- moved Y1 19.3 mm to (195.6, 105.7), turned to 0 degrees
- moved D1 14.8 mm to (169.7, 91.4)
- moved C4 13.4 mm to (161.5, 70.1), turned to 270 degrees
- moved R2 12.2 mm to (205.7, 105.2), turned to 0 degrees
- moved C1 10.2 mm to (206.8, 77.2), turned to 270 degrees
- moved C2 10.2 mm to (212.9, 87.4), turned to 90 degrees
- moved J1 8.38 mm to (178.9, 98.0)
- moved U3 4.79 mm to (182.4, 79.8)
- moved R1 4.59 mm to (169.7, 78.7)
- moved D2 2.73 mm to (169.7, 84.8)
- moved C3 2.50 mm to (161.5, 83.8), turned to 270 degrees
- moved J2 2.03 mm to (141.6, 70.1)
Connections:
- J1 pad 12: /COMPUTER_SDA -> Net-(J1-Pad12)
- J1 pad 15: /COMPUTER_SCL -> Net-(J1-Pad15)
Routing:
- net GND: track 262.0 -> 190.0 mm
- net /COMPUTER_5V: track 11.6 -> 51.4 mm
- net /H_SYNC: track 36.9 -> 66.1 mm
- net /5V_TRICKLE: track 57.2 -> 78.1 mm
- net Net-(C4-Pad1): track 25.1 -> 45.2 mm
- net /DCO: track 68.3 -> 52.3 mm
- net /RED: track 25.8 -> 39.5 mm
- net /COMPUTER_SCL: track 38.5 -> 49.5 mm, vias 1 -> 0
- net Net-(D1-Pad1): track 40.4 -> 29.5 mm
- net /COMPUTER_SDA: track 70.0 -> 59.6 mm
- net Net-(C3-Pad2): track 27.1 -> 36.8 mm
- net /BLUE: track 25.6 -> 33.8 mm, vias 1 -> 0
- net /V_SYNC: track 37.6 -> 45.5 mm
- net /GREEN: track 25.3 -> 32.1 mm
- net Net-(J1-Pad15): track 0.00 -> 5.72 mm
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Other:
- board size 82.6 x 45.9 mm -> 82.6 x 52.5 mm
- board text added: "Rocky Hill"
- board text added: "iMac G3 DV VGA on/off adapter"
- board text added: "solder jumpers to send EDID"
