File: schematics_and_pcbs/imac_g3_333mhz_slot_loading_J20_adapter_board/imac_g3_333mhz_slot_loading_J20_adapter_board.kicad_pcb (KiCad board)
At the start: 2 copper layers, 82.6 x 52.5 mm, 21 parts, among them J1 DB15_Female_HighDensity, J2 Screw_Terminal_01x06, J20 Conn_02x10_Odd_Even, U1 ATmega328-PU, U2 ATmega328-PU, U3 LCC110, Y1 Crystal, Y2 Crystal

Commit message: removed an atmega328 and moved VGA connector
Parts:
- removed the C3 at (161.5, 83.8)
- removed C4: 22pF, Capacitor_THT:C_Disc_D9.0mm_W5.0mm_P10.00mm
- removed C6: 470uF, Capacitor_THT:CP_Radial_D8.0mm_P3.50mm
- removed the J2 at (141.6, 70.1)
- removed the U2 at (149.2, 65.4)
- removed Y2: Crystal, Crystal:Crystal_HC49-U_Vertical
- added H1: MountingHole_Pad, MountingHole:MountingHole_3.5mm_Pad, F.Cu at (139.2, 69.9)
- added J3: Conn_02x03_Odd_Even, Connector_PinHeader_2.54mm:PinHeader_2x03_P2.54mm_Vertical, F.Cu at (171.2, 106.7)
- added J4: DB15_Female_HighDensity, Connector_Dsub:DSUB-15-HD_Female_Horizontal_P2.29x1.98mm_EdgePinOffset8.35mm_Housed_MountingHolesOffset10.89mm, F.Cu at (199.4, 86.4)
- added J5: Conn_02x03_Odd_Even, Connector_PinHeader_2.54mm:PinHeader_2x03_P2.54mm_Vertical, F.Cu at (180.4, 101.4)
- added R1: 10k, Resistor_THT:R_Axial_DIN0207_L6.3mm_D2.5mm_P7.62mm_Horizontal, F.Cu at (191.7, 78.4)
- added R3: 10k, Resistor_THT:R_Axial_DIN0207_L6.3mm_D2.5mm_P7.62mm_Horizontal, F.Cu at (162.7, 68.9)
- C1, C2: value 22pF -> 20pF; footprint Capacitor_THT:C_Disc_D9.0mm_W5.0mm_P10.00mm -> Capacitor_THT:C_Disc_D5.0mm_W2.5mm_P5.00mm
- J1: value DB15_Female_HighDensity -> Screw_Terminal_01x06; footprint Connector_Dsub:DSUB-15-HD_Female_Horizontal_P2.29x1.98mm_EdgePinOffset8.35mm_Housed_MountingHolesOffset10.89mm -> TerminalBlock_Phoenix:TerminalBlock_Phoenix_PT-1,5-6-5.0-H_1x06_P5.00mm_Horizontal
- JP1, JP2: moved to F.Cu
- moved C2 63.9 mm to (150.7, 102.2), turned to 270 degrees
- moved C1 56.3 mm to (150.7, 81.4)
- moved Y1 47.0 mm to (150.7, 91.9), turned to 270 degrees
- moved J1 41.4 mm to (141.6, 80.2), turned to 270 degrees
- moved U1 39.9 mm to (155.7, 74.2)
- moved R2 36.8 mm to (201.4, 68.7), turned to 180 degrees
- moved C3 23.2 mm to (185.4, 90.9)
- moved JP2 18.1 mm to (178.7, 93.2), turned to 90 degrees
- moved R4 17.8 mm to (167.9, 96.4), turned to 90 degrees
- moved D2 16.3 mm to (185.7, 81.7), turned to 90 degrees
- moved U2 15.5 mm to (167.9, 74.2)
- moved D1 14.5 mm to (180.7, 81.9), turned to 90 degrees
- moved JP1 13.6 mm to (173.2, 93.4), turned to 90 degrees
- moved H2 0.50 mm to (209.2, 70.2)
- renumbered C5 to C3, H1 to H2, J20 to J2, R1 to R4, U3 to U2
Connections:
- J1 pad 1: /RED -> /PWR_BTN
- J1 pad 2: /GREEN -> /LINE_SENSE
- J1 pad 3: /BLUE -> /-10V
- J1 pad 4: Net-(J1-Pad4) -> /PROT
- J1 pad 5: GND -> /DCO
- J1 pad 6: GND -> /LPIACT:L1_LP
- JP1 pad 1: Net-(J1-Pad12) -> Net-(J4-Pad12)
- JP2 pad 1: Net-(J1-Pad15) -> Net-(J4-Pad15)
- R2 pad 1: /PWR_BTN -> GND
- R2 pad 2: /5V_TRICKLE -> /PROT
- U1 pad 1: Net-(U1-Pad1) -> /~RESET
- U1 pad 11: Net-(U1-Pad11) -> /IVAD_SCL
- U1 pad 14: Net-(U1-Pad14) -> /PB0
- U1 pad 15: Net-(U1-Pad15) -> /PB1
- U1 pad 17: Net-(U1-Pad17) -> /MOSI
- U1 pad 18: Net-(U1-Pad18) -> /MISO
- U1 pad 19: /PWR_BTN -> /SCK
- U1 pad 2: Net-(U1-Pad2) -> /SERIAL_RX
- U1 pad 20: /5V_TRICKLE -> Net-(D1-Pad1)
- U1 pad 27: /IVAD_SDA -> /COMPUTER_SDA
- U1 pad 28: /IVAD_SCL -> /COMPUTER_SCL
- U1 pad 3: Net-(U1-Pad3) -> /SERIAL_TX
- U1 pad 5: Net-(U1-Pad5) -> /PWR_BTN
- U1 pad 6: Net-(U1-Pad6) -> /IVAD_SDA
- U1 pad 7: /5V_TRICKLE -> Net-(D1-Pad1)
Routing:
- net GND: track 190.0 -> 54.4 mm, vias 0 -> 18
- net /IVAD_SCL: track 13.9 -> 79.2 mm
- net Net-(J4-Pad12): track 0.00 -> 57.4 mm
- net /SERIAL_TX: track 0.00 -> 54.5 mm
- net /SERIAL_RX: track 0.00 -> 47.6 mm
- net Net-(C4-Pad1): track 45.2 -> 0.00 mm
- net /~RESET: track 0.00 -> 40.2 mm
- net /PWR_BTN: track 94.7 -> 54.6 mm
- net /PB0: track 0.00 -> 37.9 mm
- net /DCO: track 52.3 -> 89.3 mm, vias 0 -> 2
- net Net-(C3-Pad2): track 36.8 -> 0.00 mm
- net /PROT: track 47.1 -> 82.7 mm
- net /IVAD_SDA: track 13.9 -> 44.6 mm, vias 0 -> 1
- net /5V_TRICKLE: track 78.1 -> 106.6 mm
- net /V_SYNC: track 45.5 -> 71.9 mm
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Other:
- board size 82.6 x 52.5 mm -> 82.5 x 52.5 mm
- board text added: "14 BP0"
- board text added: "15 PB1"
- board text added: "5V"
- board text added: "MISO"
- board text added: "MOSI"
- board text added: "POWER BUTTON"
- board text added: "POWER LED"
- board text added: "SCK"
- board text added: "SENSE"
- board text added: "SERIAL RX"
- board text added: "SERIAL TX"
- board text added: "~RESET"
- board text removed: "PWR-BTN"
- board text removed: "PWR/LED"
- board text removed: "SNS"

Commit message: added resistor values to silkscreen
Other:
- board text added: "10k"
- board text added: "16 MHz"
- board text added: "20pF"
- board text added: "220"
- board text added: "470uF"
- board text added: "Yeah, cute. Don't get too attached there, Aladdin, 'cause it's about to be magic flying dinner."
Changed lines of the file:
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@@
   (general
     (thickness 1.6)
-    (drawings 50)
+    (drawings 59)
     (tracks 401)
     (zones 0)
@@
     (descr "Resistor, Axial_DIN0207 series, Axial, Horizontal, pin pitch=7.62mm, 0.25W = 1/4W, length*diameter=6.3*2.5mm^2, http://cdn-reichelt.de/documents/datenblatt/B400/1_4W%23YAG.pdf")
     (tags "Resistor Axial_DIN0207 series Axial Horizontal pin pitch 7.62mm 0.25W = 1/4W length 6.3mm diameter 2.5mm")
-    (fp_text reference R1 (at 7.112 3.048 -180) (layer F.SilkS)
+    (fp_text reference R1 (at 2.25 2.75 -180) (layer F.SilkS)
       (effects (font (size 1 1) (thickness 0.15)))
     )
@@
     (descr "Resistor, Axial_DIN0207 series, Axial, Horizontal, pin pitch=7.62mm, 0.25W = 1/4W, length*diameter=6.3*2.5mm^2, http://cdn-reichelt.de/documents/datenblatt/B400/1_4W%23YAG.pdf")
     (tags "Resistor Axial_DIN0207 series Axial Horizontal pin pitch 7.62mm 0.25W = 1/4W length 6.3mm diameter 2.5mm")
-    (fp_text reference R3 (at 3.81 -2.37) (layer F.SilkS)
+    (fp_text reference R3 (at 7 -2.5) (layer F.SilkS)
       (effects (font (size 1 1) (thickness 0.15)))
     )
@@
     )
   )
+  (gr_text "Yeah, cute. Don't get too attached there, \nAladdin, 'cause it's about to be magic flying dinner." (at 159.153 86.4038 90) (layer B.SilkS)
+    (effects (font (size 1 1) (thickness 0.15)) (justify mirror))
+  )
+  (gr_text 470uF (at 186.903 96.1538) (layer F.SilkS)
+    (effects (font (size 1 1) (thickness 0.15)))
+  )
+  (gr_text "16 MHz" (at 147.153 96.9038 90) (layer F.SilkS)
+    (effects (font (size 1 1) (thickness 0.15)))
+  )
+  (gr_text 20pF (at 148.153 104.6538 90) (layer F.SilkS)
+    (effects (font (size 1 1) (thickness 0.15)))
+  )
+  (gr_text 20pF (at 147.903 83.9038 90) (layer F.SilkS)
+    (effects (font (size 1 1) (thickness 0.15)))
+  )
+  (gr_text 220 (at 170.403 92.6538 90) (layer F.SilkS)
+    (effects (font (size 1 1) (thickness 0.15)))
+  )
+  (gr_text 10k (at 158.903 66.6538) (layer F.SilkS)
+    (effects (font (size 1 1) (thickness 0.15)))
+  )
+  (gr_text 10k (at 195.403 75.9038) (layer F.SilkS)
+    (effects (font (size 1 1) (thickness 0.15)))
+  )
+  (gr_text 10k (at 197.403 66.4038) (layer F.SilkS)
+    (effects (font (size 1 1) (thickness 0.15)))
+  )
   (gr_text VGA (at 185.653 101.0538) (layer F.SilkS)
     (effects (font (size 0.5 0.5) (thickness 0.1)))
@@
   (gr_arc (start 174.625 186.181998) (end 215.899998 64.516) (angle -37.47884973) (layer Edge.Cuts) (width 0.05))
   (gr_arc (start 134.35 109.22) (end 133.35 109.22) (angle -90) (layer Edge.Cuts) (width 0.05))
-  (gr_text VGA (at 182.88 86.36) (layer F.SilkS)
+  (gr_text VGA (at 196.653 84.6538 60) (layer F.SilkS)
     (effects (font (size 1 1) (thickness 0.15)))
   )
@@
   (segment (start 187.9276 68.472) (end 186.724399 69.675201) (width 0.25) (layer B.Cu) (net 9))
   (segment (start 199.3975 94.3334) (end 200.162 94.3334) (width 0.25) (layer B.Cu) (net 10))
-  (segment (start 194.6348 64.3856) (end 197.003001 66.753801) (width 0.25) (layer F.Cu) (net 10))
   (segment (start 176.403 68.1038) (end 177.5783 66.9285) (width 0.25) (layer F.Cu) (net 10))
   (via (at 197.403 67.1538) (size 0.8) (drill 0.4) (layers F.Cu B.Cu) (net 10))
@@
   (segment (start 179.3394 66.9285) (end 180.3076 65.9603) (width 0.25) (layer F.Cu) (net 10))
   (segment (start 180.3076 65.9603) (end 180.3076 65.0283) (width 0.25) (layer F.Cu) (net 10))
+  (segment (start 180.9503 64.3856) (end 194.6348 64.3856) (width 0.25) (layer F.Cu) (net 10))
+  (segment (start 213.702989 79.453789) (end 209.702989 79.453789) (width 0.25) (layer B.Cu) (net 10))
+  (segment (start 205.473405 94.333395) (end 213.238566 86.568234) (width 0.25) (layer B.Cu) (net 10))
+  (segment (start 215.549988 82.560112) (end 215.549988 81.300788) (width 0.25) (layer B.Cu) (net 10))
+  (segment (start 199.397461 94.333395) (end 205.473405 94.333395) (width 0.25) (layer B.Cu) (net 10))
+  (segment (start 213.238566 86.568234) (end 215.549988 82.560112) (width 0.25) (layer B.Cu) (net 10))
+  (segment (start 215.549988 81.300788) (end 213.702989 79.453789) (width 0.25) (layer B.Cu) (net 10))
+  (segment (start 209.702989 79.453789) (end 197.802999 67.553799) (width 0.25) (layer B.Cu) (net 10))
+  (segment (start 197.802999 67.553799) (end 197.403 67.1538) (width 0.25) (layer B.Cu) (net 10))
+  (segment (start 194.6348 64.3856) (end 197.003001 66.753801) (width 0.25) (layer F.Cu) (net 10))
   (segment (start 197.003001 66.753801) (end 197.403 67.1538) (width 0.25) (layer F.Cu) (net 10))
-  (segment (start 180.9503 64.3856) (end 194.6348 64.3856) (width 0.25) (layer F.Cu) (net 10))
-  (segment (start 197.802999 67.553799) (end 197.403 67.1538) (width 0.25) (layer B.Cu) (net 10))
-  (segment (start 205.473405 94.333395) (end 213.238566 86.568234) (width 0.25) (layer B.Cu) (net 10))
-  (segment (start 209.702989 79.453789) (end 197.802999 67.553799) (width 0.25) (layer B.Cu) (net 10))
-  (segment (start 199.397461 94.333395) (end 205.473405 94.333395) (width 0.25) (layer B.Cu) (net 10))
-  (segment (start 215.549988 81.300788) (end 213.702989 79.453789) (width 0.25) (layer B.Cu) (net 10))
-  (segment (start 213.238566 86.568234) (end 215.549988 82.560112) (width 0.25) (layer B.Cu) (net 10))
-  (segment (start 215.549988 82.560112) (end 215.549988 81.300788) (width 0.25) (layer B.Cu) (net 10))
-  (segment (start 213.702989 79.453789) (end 209.702989 79.453789) (width 0.25) (layer B.Cu) (net 10))
   (segment (start 168.082 75.2791) (end 169.3832 76.5803) (width 0.25) (layer B.Cu) (net 11))
   (segment (start 164.3983 75.2791) (end 168.082 75.2791) (width 0.25) (layer B.Cu) (net 11))

Commit message: updated silkscreen to make it more readable
Other:
- board text added: "ICSP"
- board text added: "PWR BUTTON"
- board text added: "PWR LED"
- board text added: "VGA SCL"
- board text added: "VGA SDA"
- board text removed: "POWER BUTTON"
- board text removed: "POWER LED"
Changed lines of the file:
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@@
   (general
     (thickness 1.6)
-    (drawings 59)
+    (drawings 63)
     (tracks 401)
     (zones 0)
@@
     (31 B.Cu signal)
     (32 B.Adhes user)
-    (33 F.Adhes user hide)
+    (33 F.Adhes user)
     (34 B.Paste user)
     (35 F.Paste user)
@@
     (descr "Through hole straight pin header, 2x03, 2.54mm pitch, double rows")
     (tags "Through hole pin header THT 2x03 2.54mm double row")
-    (fp_text reference J3 (at 1.27 -2.33) (layer F.SilkS)
+    (fp_text reference J3 (at 1.5 7.7502) (layer F.SilkS)
       (effects (font (size 1 1) (thickness 0.15)))
     )
@@
     )
   )
+  (gr_line (start 135.903 82.9038) (end 133.653 82.9038) (layer F.SilkS) (width 0.12))
+  (gr_line (start 135.903 88.1538) (end 133.653 88.1538) (layer F.SilkS) (width 0.12))
+  (gr_line (start 135.903 92.1538) (end 133.653 92.1538) (layer F.SilkS) (width 0.12))
+  (gr_line (start 135.903 97.6538) (end 133.653 97.6538) (layer F.SilkS) (width 0.12))
+  (gr_line (start 135.903 102.9038) (end 133.653 102.9038) (layer F.SilkS) (width 0.12))
+  (gr_text ICSP (at 169.903 109.4038) (layer F.SilkS)
+    (effects (font (size 1 1) (thickness 0.15)))
+  )
   (gr_text "Yeah, cute. Don't get too attached there, \nAladdin, 'cause it's about to be magic flying dinner." (at 159.153 86.4038 90) (layer B.SilkS)
     (effects (font (size 1 1) (thickness 0.15)) (justify mirror))
@@
     (effects (font (size 1 1) (thickness 0.15)))
   )
-  (gr_text VGA (at 185.653 101.0538) (layer F.SilkS)
-    (effects (font (size 0.5 0.5) (thickness 0.1)))
-  )
-  (gr_text VGA (at 177.853 101.0538) (layer F.SilkS)
-    (effects (font (size 0.5 0.5) (thickness 0.1)))
-  )
-  (gr_text "14\nBP0" (at 185.653 103.9038) (layer F.SilkS)
-    (effects (font (size 0.5 0.5) (thickness 0.1)))
-  )
-  (gr_text "15\nPB1" (at 185.653 106.9038) (layer F.SilkS)
-    (effects (font (size 0.5 0.5) (thickness 0.1)))
-  )
-  (gr_text SCL (at 185.653 101.7538) (layer F.SilkS)
-    (effects (font (size 0.5 0.5) (thickness 0.1)))
-  )
-  (gr_text "SERIAL\nTX" (at 177.153 106.9038) (layer F.SilkS)
-    (effects (font (size 0.5 0.5) (thickness 0.1)))
-  )
-  (gr_text SDA (at 177.853 101.8038) (layer F.SilkS)
-    (effects (font (size 0.5 0.5) (thickness 0.1)))
-  )
-  (gr_text "SERIAL\nRX" (at 177.153 104.1538) (layer F.SilkS)
-    (effects (font (size 0.5 0.5) (thickness 0.1)))
-  )
-  (gr_text 5V (at 165.703 106.9538) (layer F.SilkS)
-    (effects (font (size 0.5 0.5) (thickness 0.1)))
-  )
-  (gr_text MOSI (at 165.703 104.2038) (layer F.SilkS)
-    (effects (font (size 0.5 0.5) (thickness 0.1)))
-  )
-  (gr_text GND (at 165.753 101.5538) (layer F.SilkS)
-    (effects (font (size 0.5 0.5) (thickness 0.1)))
-  )
-  (gr_text MISO (at 174.253 106.9538) (layer F.SilkS)
-    (effects (font (size 0.5 0.5) (thickness 0.1)))
-  )
-  (gr_text SCK (at 174.103 104.2538) (layer F.SilkS)
-    (effects (font (size 0.5 0.5) (thickness 0.1)))
-  )
-  (gr_text ~RESET (at 174.303 101.7038) (layer F.SilkS)
-    (effects (font (size 0.5 0.5) (thickness 0.1)))
+  (gr_text "VGA\nSCL" (at 185.903 100.4038) (layer F.SilkS)
+    (effects (font (size 0.8 0.8) (thickness 0.15)))
+  )
+  (gr_text "VGA\nSDA" (at 177.653 100.4038) (layer F.SilkS)
+    (effects (font (size 0.7 0.7) (thickness 0.15)))
+  )
+  (gr_text "14\nBP0" (at 186.153 103.9038) (layer F.SilkS)
+    (effects (font (size 0.8 0.8) (thickness 0.15)))
+  )
+  (gr_text "15\nPB1" (at 186.153 106.9038) (layer F.SilkS)
+    (effects (font (size 0.8 0.8) (thickness 0.15)))
+  )
+  (gr_text "SERIAL\nTX" (at 176.903 107.4038) (layer F.SilkS)
+    (effects (font (size 0.7 0.7) (thickness 0.15)))
+  )
+  (gr_text "SERIAL\nRX" (at 176.903 103.9038) (layer F.SilkS)
+    (effects (font (size 0.7 0.7) (thickness 0.15)))
+  )
+  (gr_text 5V (at 166.153 107.1538 90) (layer F.SilkS)
+    (effects (font (size 0.8 0.8) (thickness 0.15)))
+  )
+  (gr_text MOSI (at 166.153 104.2038 90) (layer F.SilkS)
+    (effects (font (size 0.8 0.8) (thickness 0.15)))
+  )
+  (gr_text GND (at 166.153 100.9038 90) (layer F.SilkS)
+    (effects (font (size 0.8 0.8) (thickness 0.15)))
+  )
+  (gr_text MISO (at 173.653 107.4038 90) (layer F.SilkS)
+    (effects (font (size 0.8 0.8) (thickness 0.15)))
+  )
+  (gr_text SCK (at 173.653 104.1538 90) (layer F.SilkS)
+    (effects (font (size 0.8 0.8) (thickness 0.15)))
+  )
+  (gr_text ~RESET (at 173.903 100.9038 90) (layer F.SilkS)
+    (effects (font (size 0.7 0.7) (thickness 0.15)))
   )
   (gr_line (start 200.003 110.22) (end 134.35 110.22) (layer Edge.Cuts) (width 0.05))
@@
     (effects (font (size 1 1) (thickness 0.15)))
   )
-  (gr_text "solder jumpers to\nsend EDID" (at 176.903 89.6538) (layer F.SilkS)
-    (effects (font (size 0.5 0.5) (thickness 0.1)))
+  (gr_text "solder jumpers to\nsend EDID" (at 176.103 89.3038) (layer F.SilkS)
+    (effects (font (size 1 1) (thickness 0.15)))
   )
   (gr_line (start 133.35 109.22) (end 133.35 64.516001) (layer Edge.Cuts) (width 0.05))
-  (gr_text "POWER\nLED" (at 134.9 106.012 90) (layer F.SilkS)
-    (effects (font (size 0.5 0.5) (thickness 0.1)))
-  )
-  (gr_text "POWER\nBUTTON" (at 134.9 80.236 90) (layer F.SilkS)
-    (effects (font (size 0.5 0.5) (thickness 0.1)))
-  )
-  (gr_text SENSE (at 134.112 85.184 90) (layer F.SilkS)
-    (effects (font (size 0.5 0.5) (thickness 0.1)))
+  (gr_text "PWR\nLED" (at 134.9 106.012 90) (layer F.SilkS)
+    (effects (font (size 0.8 0.8) (thickness 0.15)))
+  )
+  (gr_text "PWR\nBUTTON" (at 134.9 80.236 90) (layer F.SilkS)
+    (effects (font (size 0.8 0.8) (thickness 0.15)))
+  )
+  (gr_text SENSE (at 134.112 85.6538 90) (layer F.SilkS)
+    (effects (font (size 0.8 0.8) (thickness 0.15)))
   )
   (gr_text DCO (at 134.112 99.916 90) (layer F.SilkS)
-    (effects (font (size 0.5 0.5) (thickness 0.1)))
+    (effects (font (size 0.8 0.8) (thickness 0.15)))
   )
   (gr_text PROT (at 134.112 95.344 90) (layer F.SilkS)
-    (effects (font (size 0.5 0.5) (thickness 0.1)))
+    (effects (font (size 0.8 0.8) (thickness 0.15)))
   )
   (gr_text -10V (at 134.112 90.264 90) (layer F.SilkS)
-    (effects (font (size 0.5 0.5) (thickness 0.1)))
+    (effects (font (size 0.8 0.8) (thickness 0.15)))
   )
   (gr_arc (start 174.625 186.181998) (end 215.899998 64.516) (angle -37.47884973) (layer Edge.Cuts) (width 0.05))

Commit message: updated schematic with a VSYNC detect input line.
Parts:
- added JP3: SolderJumper_2_Open, Jumper:SolderJumper-2_P1.3mm_Open_RoundedPad1.0x1.5mm, F.Cu at (150.7, 73.9)
- C1, C2: value 20pF -> 22pF
Routing:
- net Net-(JP3-Pad1): track 0.00 -> 47.3 mm, vias 0 -> 2
- net /V_SYNC: track 71.9 -> 108.0 mm, vias 1 -> 5
Other:
- board text added: "Rev 3"
- board text added: "SOLDER JP3 TO USE VSYNC DETECT"
