File: schematics_and_pcbs/imac_g3_333mhz_slot_loading_J20_adapter_board/imac_g3_333mhz_slot_loading_J20_adapter_board.sch (KiCad schematic (older format))
At the start: 10 parts, among them J20 Conn_02x10_Odd_Even

Commit message: updated schematic with new J20 info
Connections:
- net labels added: -10V, 5V_TRICKLE, DCO, LINE_SENSE, LPIACT:L1_LP, PROT
- net labels removed: +5V, 40V, 50V_1, 50V_2, 50V_3, 50V_4, PFW_5V
- wire segments 73 -> 79
- no-connect marks 6 -> 4
Other:
- note added: "Sends EDID data to computer via DE15\nconnector"
- note added: "Sends initialization sequence to the IVAD board"
Changed lines of the file:
@@
 Comp ""
 Comment1 "and control other functions."
-Comment2 "used to send the i2c IVAD inititialization sequence"
-Comment3 "Converts 50 Volts DC fromJ20 to power an atmega328p"
+Comment2 "used to send the i2c IVAD inititialization sequence and the EDID info to the computer"
+Comment3 "Powers atmega328p fromJ20 and powers an atmega328p from VGA cable"
 Comment4 "Rocky Hill"
 $EndDescr
@@
 	1    0    0    -1
 $EndComp
-$Comp
-L power:+5V #PWR?
-U 1 1 5E398311
-P 1400 850
-F 0 "#PWR?" H 1400 700 50  0001 C CNN
-F 1 "+5V" H 1415 1023 50  0000 C CNN
-F 2 "" H 1400 850 50  0001 C CNN
-F 3 "" H 1400 850 50  0001 C CNN
-	1    1400 850
-	1    0    0    -1
-$EndComp
 Wire Wire Line
 	1350 1150 1350 850
 Wire Wire Line
-	1350 850  1400 850
-Wire Wire Line
 	1450 1150 1450 850
-Wire Wire Line
-	1450 850  1400 850
-Connection ~ 1400 850
 NoConn ~ 750  1450
 $Comp
@@
 	9200 1900 9600 1900
 Text Label 9600 1300 0    50   ~ 0
-PFW_5V
+5V_TRICKLE
 Wire Wire Line
 	9200 1300 9600 1300
-NoConn ~ 9200 2000
-NoConn ~ 8700 2000
-$Comp
-L Connector_Generic:Conn_02x10_Odd_Even J20
-U 1 1 5E3F686C
-P 8900 1500
-F 0 "J20" H 8950 2117 50  0000 C CNN
-F 1 "Conn_02x10_Odd_Even" H 8950 2026 50  0000 C CNN
-F 2 "" H 8900 1500 50  0001 C CNN
-F 3 "~" H 8900 1500 50  0001 C CNN
-	1    8900 1500
-	1    0    0    -1
-$EndComp
 $Comp
 L MCU_Microchip_ATmega:ATmega328-PU U?
@@
 	1    0    0    -1
 $EndComp
-$Comp
-L power:+5V #PWR?
-U 1 1 5E42FE51
-P 4300 3950
-F 0 "#PWR?" H 4300 3800 50  0001 C CNN
-F 1 "+5V" H 4315 4123 50  0000 C CNN
-F 2 "" H 4300 3950 50  0001 C CNN
-F 3 "" H 4300 3950 50  0001 C CNN
-	1    4300 3950
-	1    0    0    -1
-$EndComp
 Wire Wire Line
 	4250 4250 4250 3950
 Wire Wire Line
-	4250 3950 4300 3950
-Wire Wire Line
 	4350 4250 4350 3950
-Wire Wire Line
-	4350 3950 4300 3950
-Connection ~ 4300 3950
 NoConn ~ 3650 4550
 $Comp
@@
 	1    0    0    -1
 $EndComp
-Text Label 9600 1200 0    50   ~ 0
-50V_1
+Text Label 8300 1400 2    50   ~ 0
+PROT
+Text Label 9600 1400 0    50   ~ 0
+-10V
+Text Label 9600 1600 0    50   ~ 0
+LPIACT:L1_LP
+Wire Wire Line
+	8700 1300 8300 1300
+Wire Wire Line
+	9200 1100 9600 1100
+Wire Wire Line
+	9200 1400 9600 1400
+Wire Wire Line
+	8700 1400 8300 1400
+Wire Wire Line
+	9600 1600 9200 1600
+$Comp
+L power:GND #PWR?
+U 1 1 5E4745C4
+P 10300 2100
+F 0 "#PWR?" H 10300 1850 50  0001 C CNN
+F 1 "GND" H 10305 1927 50  0000 C CNN
+F 2 "" H 10300 2100 50  0001 C CNN
+F 3 "" H 10300 2100 50  0001 C CNN
+	1    10300 2100
+	1    0    0    -1
+$EndComp
 Text Label 8300 1300 2    50   ~ 0
-50V_2
-Text Label 8300 1400 2    50   ~ 0
-50V_3
-Text Label 9600 1400 0    50   ~ 0
-40V
-Text Label 9600 1600 0    50   ~ 0
-50V_4
-Wire Wire Line
-	8700 1300 8300 1300
-Wire Wire Line
-	9200 1100 9600 1100
-Wire Wire Line
-	9600 1200 9200 1200
-Wire Wire Line
-	9200 1400 9600 1400
-Wire Wire Line
-	8700 1400 8300 1400
-Wire Wire Line
-	9600 1600 9200 1600
+DCO
+$Comp
+L Connector_Generic:Conn_02x10_Odd_Even J20
+U 1 1 5E3F686C
+P 8900 1500
+F 0 "J20" H 8950 2117 50  0000 C CNN
+F 1 "Conn_02x10_Odd_Even" H 8950 2026 50  0000 C CNN
+F 2 "" H 8900 1500 50  0001 C CNN
+F 3 "~" H 8900 1500 50  0001 C CNN
+	1    8900 1500
+	1    0    0    -1
+$EndComp
+Text Label 8300 2000 2    50   ~ 0
+LINE_SENSE
+Wire Wire Line
+	10300 1200 10300 2000
+Wire Wire Line
+	9200 1200 10300 1200
+Wire Wire Line
+	9200 2000 10300 2000
+Connection ~ 10300 2000
+Wire Wire Line
+	10300 2000 10300 2100
+Wire Wire Line
+	8700 2000 8300 2000
+Wire Wire Line
+	1350 850  1400 850
+Text Label 1400 700  0    50   ~ 0
+5V_TRICKLE
+Wire Wire Line
+	1400 700  1400 850
+Connection ~ 1400 850
+Wire Wire Line
+	1400 850  1450 850
+Wire Wire Line
+	4250 3950 4300 3950
+Text Label 4300 3750 0    50   ~ 0
+COMPUTER_5V
+Wire Wire Line
+	4300 3750 4300 3950
+Connection ~ 4300 3950
+Wire Wire Line
+	4300 3950 4350 3950
+Text Notes 900  4800 0    50   ~ 0
+Sends initialization sequence to the IVAD board
+Text Notes 2100 6550 0    50   ~ 0
+Sends EDID data to computer via DE15\nconnector
 $EndSCHEMATC

Commit message: made a test pcb
Parts:
- removed C? (x3): C, symbol Device:C
- removed Y?: Crystal, symbol Device:Crystal
- added C2, C3, C4: 22pF, Capacitor_THT:C_Disc_D9.0mm_W5.0mm_P10.00mm, symbol Device:C
- added H1, H2: MountingHole, MountingHole:MountingHole_3.5mm_Pad, symbol Mechanical:MountingHole
- added Y2: Crystal, Crystal:Crystal_HC49-U_Vertical, symbol Device:Crystal
- C1: renamed from C?; value C -> 22pF; footprint (none) -> Capacitor_THT:C_Disc_D9.0mm_W5.0mm_P10.00mm; Part# (none) -> BC2364-ND; Vendor (none) -> digikey
- J1: renamed from J?; footprint (none) -> Connector_Dsub:DSUB-15-HD_Female_Horizontal_P2.29x1.98mm_EdgePinOffset8.35mm_Housed_MountingHolesOffset10.89mm; Part# (none) -> L77HDE15SD1CH4F-ND; Vendor (none) -> digikey
- J20: footprint (none) -> Connector_PinHeader_2.54mm:PinHeader_2x10_P2.54mm_Vertical; Part# (none) -> 609-2430-ND; Vendor (none) -> digikey
- Y1: renamed from Y?; footprint (none) -> Crystal:Crystal_HC49-U_Vertical; Part# (none) -> 887-2015-ND; Vendor (none) -> digikey
- gave numbers to parts that had none: 2
Connections:
- net GND: now also C2.2, C3.1, C4.2
- net at U1.10 (XTAL2/PB7), Y1.2: now also C2.1
- net at U2.10 (XTAL2/PB7): now also C4.1, Y2.2
- net at U2.9 (XTAL1/PB6): now also C3.2, Y2.1
Changed lines of the file:
@@
 $EndDescr
 $Comp
-L MCU_Microchip_ATmega:ATmega328-PU U?
+L MCU_Microchip_ATmega:ATmega328-PU U1
 U 1 1 5E393326
 P 1350 2650
-F 0 "U?" H 1100 4250 50  0000 R CNN
+F 0 "U1" H 1100 4250 50  0000 R CNN
 F 1 "ATmega328-PU" H 2250 4350 50  0000 R CNN
 F 2 "Package_DIP:DIP-28_W7.62mm" H 1350 2650 50  0001 C CIN
@@
 NoConn ~ 750  1450
 $Comp
-L power:GND #PWR?
+L power:GND #PWR07
 U 1 1 5E39A336
 P 1350 4450
-F 0 "#PWR?" H 1350 4200 50  0001 C CNN
+F 0 "#PWR07" H 1350 4200 50  0001 C CNN
 F 1 "GND" H 1355 4277 50  0000 C CNN
 F 2 "" H 1350 4450 50  0001 C CNN
@@
 	1350 4150 1350 4450
 $Comp
-L Device:Crystal Y?
+L Device:Crystal Y1
 U 1 1 5E39C3FD
 P 3400 2100
-F 0 "Y?" V 3354 2231 50  0000 L CNN
+F 0 "Y1" V 3354 2231 50  0000 L CNN
 F 1 "Crystal" V 3445 2231 50  0000 L CNN
-F 2 "" H 3400 2100 50  0001 C CNN
-F 3 "~" H 3400 2100 50  0001 C CNN
+F 2 "Crystal:Crystal_HC49-U_Vertical" H 3400 2100 50  0001 C CNN
+F 3 "http://www.txccrystal.com/images/pdf/9b.pdf" H 3400 2100 50  0001 C CNN
+F 4 "digikey" V 3400 2100 50  0001 C CNN "Vendor"
+F 5 "887-2015-ND" V 3400 2100 50  0001 C CNN "Part#"
 	1    3400 2100
 	0    1    1    0
 $EndComp
 $Comp
-L Device:C C?
+L Device:C C1
 U 1 1 5E39D342
 P 3400 1400
-F 0 "C?" H 3515 1446 50  0000 L CNN
-F 1 "C" H 3515 1355 50  0000 L CNN
-F 2 "" H 3438 1250 50  0001 C CNN
-F 3 "~" H 3400 1400 50  0001 C CNN
+F 0 "C1" H 3515 1446 50  0000 L CNN
+F 1 "22pF" H 3515 1355 50  0000 L CNN
+F 2 "Capacitor_THT:C_Disc_D9.0mm_W5.0mm_P10.00mm" H 3438 1250 50  0001 C CNN
+F 3 "http://www.vishay.com/docs/28537/vy1series.pdf" H 3400 1400 50  0001 C CNN
+F 4 "digikey" H 3400 1400 50  0001 C CNN "Vendor"
+F 5 "BC2364-ND" H 3400 1400 50  0001 C CNN "Part#"
 	1    3400 1400
-	1    0    0    -1
-$EndComp
-$Comp
-L Device:C C?
-U 1 1 5E39DAA6
-P 3400 2800
-F 0 "C?" H 3515 2846 50  0000 L CNN
-F 1 "C" H 3515 2755 50  0000 L CNN
-F 2 "" H 3438 2650 50  0001 C CNN
-F 3 "~" H 3400 2800 50  0001 C CNN
-	1    3400 2800
 	1    0    0    -1
 $EndComp
@@
 	1950 2050 2650 2050
 $Comp
-L power:GND #PWR?
+L power:GND #PWR04
 U 1 1 5E3A7604
 P 3400 2950
-F 0 "#PWR?" H 3400 2700 50  0001 C CNN
+F 0 "#PWR04" H 3400 2700 50  0001 C CNN
 F 1 "GND" H 3405 2777 50  0000 C CNN
 F 2 "" H 3400 2950 50  0001 C CNN
@@
 $EndComp
 $Comp
-L power:GND #PWR?
+L power:GND #PWR02
 U 1 1 5E3A84E9
 P 7650 1300
-F 0 "#PWR?" H 7650 1050 50  0001 C CNN
+F 0 "#PWR02" H 7650 1050 50  0001 C CNN
 F 1 "GND" H 7655 1127 50  0000 C CNN
 F 2 "" H 7650 1300 50  0001 C CNN
@@
 	9600 1500 9200 1500
 $Comp
-L power:GND #PWR?
+L power:GND #PWR01
 U 1 1 5E3B5B7F
 P 2950 1050
-F 0 "#PWR?" H 2950 800 50  0001 C CNN
+F 0 "#PWR01" H 2950 800 50  0001 C CNN
 F 1 "GND" H 2955 877 50  0000 C CNN
 F 2 "" H 2950 1050 50  0001 C CNN
@@
 $EndComp
 $Comp
-L Connector:DB15_Female_HighDensity J?
+L Connector:DB15_Female_HighDensity J1
 U 1 1 5E3B898B
 P 8950 3400
-F 0 "J?" H 8950 4267 50  0000 C CNN
+F 0 "J1" H 8950 4267 50  0000 C CNN
 F 1 "DB15_Female_HighDensity" H 8950 4176 50  0000 C CNN
-F 2 "" H 8000 3800 50  0001 C CNN
-F 3 " ~" H 8000 3800 50  0001 C CNN
+F 2 "Connector_Dsub:DSUB-15-HD_Female_Horizontal_P2.29x1.98mm_EdgePinOffset8.35mm_Housed_MountingHolesOffset10.89mm" H 8000 3800 50  0001 C CNN
+F 3 "https://cdn.amphenol-icc.com/media/wysiwyg/files/drawing/l77hdxxxsd1ch4f.pdf" H 8000 3800 50  0001 C CNN
+F 4 "digikey" H 8950 3400 50  0001 C CNN "Vendor"
+F 5 "L77HDE15SD1CH4F-ND" H 8950 3400 50  0001 C CNN "Part#"
 	1    8950 3400
 	1    0    0    -1
@@
 NoConn ~ 8650 3600
 $Comp
-L power:GND #PWR?
+L power:GND #PWR05
 U 1 1 5E3D17A3
 P 8400 3800
-F 0 "#PWR?" H 8400 3550 50  0001 C CNN
+F 0 "#PWR05" H 8400 3550 50  0001 C CNN
 F 1 "GND" H 8405 3627 50  0000 C CNN
 F 2 "" H 8400 3800 50  0001 C CNN
@@
 	9200 1300 9600 1300
 $Comp
-L MCU_Microchip_ATmega:ATmega328-PU U?
+L MCU_Microchip_ATmega:ATmega328-PU U2
 U 1 1 5E42FE47
 P 4250 5750
-F 0 "U?" H 4000 7350 50  0000 R CNN
+F 0 "U2" H 4000 7350 50  0000 R CNN
 F 1 "ATmega328-PU" H 5150 7450 50  0000 R CNN
 F 2 "Package_DIP:DIP-28_W7.62mm" H 4250 5750 50  0001 C CIN
@@
 NoConn ~ 3650 4550
 $Comp
-L power:GND #PWR?
+L power:GND #PWR09
 U 1 1 5E42FE61
 P 4250 7550
-F 0 "#PWR?" H 4250 7300 50  0001 C CNN
+F 0 "#PWR09" H 4250 7300 50  0001 C CNN
 F 1 "GND" H 4255 7377 50  0000 C CNN
 F 2 "" H 4250 7550 50  0001 C CNN
@@
 Wire Wire Line
 	4250 7250 4250 7550
-$Comp
-L Device:Crystal Y?
-U 1 1 5E42FE6C
-P 6300 5200
-F 0 "Y?" V 6254 5331 50  0000 L CNN
-F 1 "Crystal" V 6345 5331 50  0000 L CNN
-F 2 "" H 6300 5200 50  0001 C CNN
-F 3 "~" H 6300 5200 50  0001 C CNN
-	1    6300 5200
-	0    1    1    0
-$EndComp
-$Comp
-L Device:C C?
-U 1 1 5E42FE76
-P 6300 4500
-F 0 "C?" H 6415 4546 50  0000 L CNN
-F 1 "C" H 6415 4455 50  0000 L CNN
-F 2 "" H 6338 4350 50  0001 C CNN
-F 3 "~" H 6300 4500 50  0001 C CNN
-	1    6300 4500
-	1    0    0    -1
-$EndComp
-$Comp
-L Device:C C?
-U 1 1 5E42FE80
-P 6300 5900
-F 0 "C?" H 6415 5946 50  0000 L CNN
-F 1 "C" H 6415 5855 50  0000 L CNN
-F 2 "" H 6338 5750 50  0001 C CNN
-F 3 "~" H 6300 5900 50  0001 C CNN
-	1    6300 5900
-	1    0    0    -1
-$EndComp
 Wire Wire Line
 	6300 4650 6300 4850
@@
 	4850 5150 5550 5150
 $Comp
-L power:GND #PWR?
+L power:GND #PWR08
 U 1 1 5E42FE96
 P 6300 6050
-F 0 "#PWR?" H 6300 5800 50  0001 C CNN
+F 0 "#PWR08" H 6300 5800 50  0001 C CNN
 F 1 "GND" H 6305 5877 50  0000 C CNN
 F 2 "" H 6300 6050 50  0001 C CNN
@@
 	4850 5950 5100 5950
 $Comp
-L power:GND #PWR?
+L power:GND #PWR06
 U 1 1 5E42FEA7
 P 5850 4150
-F 0 "#PWR?" H 5850 3900 50  0001 C CNN
+F 0 "#PWR06" H 5850 3900 50  0001 C CNN
 F 1 "GND" H 5855 3977 50  0000 C CNN
 F 2 "" H 5850 4150 50  0001 C CNN
@@
 	9600 1600 9200 1600
 $Comp
-L power:GND #PWR?
+L power:GND #PWR03
 U 1 1 5E4745C4
 P 10300 2100
-F 0 "#PWR?" H 10300 1850 50  0001 C CNN
+F 0 "#PWR03" H 10300 1850 50  0001 C CNN
 F 1 "GND" H 10305 1927 50  0000 C CNN
 F 2 "" H 10300 2100 50  0001 C CNN
@@
 F 0 "J20" H 8950 2117 50  0000 C CNN
 F 1 "Conn_02x10_Odd_Even" H 8950 2026 50  0000 C CNN
-F 2 "" H 8900 1500 50  0001 C CNN
-F 3 "~" H 8900 1500 50  0001 C CNN
+F 2 "Connector_PinHeader_2.54mm:PinHeader_2x10_P2.54mm_Vertical" H 8900 1500 50  0001 C CNN
+F 3 "https://cdn.amphenol-icc.com/media/wysiwyg/files/drawing/69168.pdf" H 8900 1500 50  0001 C CNN
+F 4 "digikey" H 8900 1500 50  0001 C CNN "Vendor"
+F 5 "609-2430-ND" H 8900 1500 50  0001 C CNN "Part#"
 	1    8900 1500
 	1    0    0    -1
@@
 Text Notes 2100 6550 0    50   ~ 0
 Sends EDID data to computer via DE15\nconnector
+$Comp
+L Device:C C2
+U 1 1 5E552ABD
+P 3400 2800
+F 0 "C2" H 3515 2846 50  0000 L CNN
+F 1 "22pF" H 3515 2755 50  0000 L CNN
+F 2 "Capacitor_THT:C_Disc_D9.0mm_W5.0mm_P10.00mm" H 3438 2650 50  0001 C CNN
+F 3 "http://www.vishay.com/docs/28537/vy1series.pdf" H 3400 2800 50  0001 C CNN
+F 4 "digikey" H 3400 2800 50  0001 C CNN "Vendor"
+F 5 "BC2364-ND" H 3400 2800 50  0001 C CNN "Part#"
+	1    3400 2800
+	1    0    0    -1
+$EndComp
+$Comp
+L Device:C C3
+U 1 1 5E552F81
+P 6300 4500
+F 0 "C3" H 6415 4546 50  0000 L CNN
+F 1 "22pF" H 6415 4455 50  0000 L CNN
+F 2 "Capacitor_THT:C_Disc_D9.0mm_W5.0mm_P10.00mm" H 6338 4350 50  0001 C CNN
+F 3 "http://www.vishay.com/docs/28537/vy1series.pdf" H 6300 4500 50  0001 C CNN
+F 4 "digikey" H 6300 4500 50  0001 C CNN "Vendor"
+F 5 "BC2364-ND" H 6300 4500 50  0001 C CNN "Part#"
+	1    6300 4500
+	1    0    0    -1
+$EndComp
+$Comp
+L Device:C C4
+U 1 1 5E554B25
+P 6300 5900
+F 0 "C4" H 6415 5946 50  0000 L CNN
+F 1 "22pF" H 6415 5855 50  0000 L CNN
+F 2 "Capacitor_THT:C_Disc_D9.0mm_W5.0mm_P10.00mm" H 6338 5750 50  0001 C CNN
+F 3 "http://www.vishay.com/docs/28537/vy1series.pdf" H 6300 5900 50  0001 C CNN
+F 4 "digikey" H 6300 5900 50  0001 C CNN "Vendor"
+F 5 "BC2364-ND" H 6300 5900 50  0001 C CNN "Part#"
+	1    6300 5900
+	1    0    0    -1
+$EndComp
+$Comp
+L Device:Crystal Y2
+U 1 1 5E555ABD
+P 6300 5200
+F 0 "Y2" V 6254 5331 50  0000 L CNN
+F 1 "Crystal" V 6345 5331 50  0000 L CNN
+F 2 "Crystal:Crystal_HC49-U_Vertical" H 6300 5200 50  0001 C CNN
+F 3 "http://www.txccrystal.com/images/pdf/9b.pdf" H 6300 5200 50  0001 C CNN
+F 4 "digikey" V 6300 5200 50  0001 C CNN "Vendor"
+F 5 "887-2015-ND" V 6300 5200 50  0001 C CNN "Part#"
+	1    6300 5200
+	0    1    1    0
+$EndComp
+$Comp
+L Mechanical:MountingHole H1
+U 1 1 5E55AF97
+P 5100 1400
+F 0 "H1" H 5200 1446 50  0000 L CNN
+F 1 "MountingHole" H 5200 1355 50  0000 L CNN
+F 2 "MountingHole:MountingHole_3.5mm_Pad" H 5100 1400 50  0001 C CNN
+F 3 "~" H 5100 1400 50  0001 C CNN
+	1    5100 1400
+	1    0    0    -1
+$EndComp
+$Comp
+L Mechanical:MountingHole H2
+U 1 1 5E55BA96
+P 5250 2200
+F 0 "H2" H 5350 2246 50  0000 L CNN
+F 1 "MountingHole" H 5350 2155 50  0000 L CNN
+F 2 "MountingHole:MountingHole_3.5mm_Pad" H 5250 2200 50  0001 C CNN
+F 3 "~" H 5250 2200 50  0001 C CNN
+	1    5250 2200
+	1    0    0    -1
+$EndComp
 $EndSCHEMATC

Commit message: made more changes to the board
Parts:
- removed H1, H2: MountingHole, MountingHole:MountingHole_3.5mm_Pad, symbol Mechanical:MountingHole
- added D1, D2: D_Schottky_ALT, Diode_THT:D_DO-41_SOD81_P7.62mm_Horizontal, symbol Device:D_Schottky_ALT
- added H1: MountingHole_Pad, MountingHole:MountingHole_3.5mm_Pad, symbol Mechanical:MountingHole_Pad
- added J2: Screw_Terminal_01x06, TerminalBlock_Phoenix:TerminalBlock_Phoenix_PT-1,5-6-5.0-H_1x06_P5.00mm_Horizontal, symbol Connector:Screw_Terminal_01x06
- added R1: 220, Resistor_THT:R_Axial_DIN0207_L6.3mm_D2.5mm_P7.62mm_Horizontal, symbol Device:R_Small_US
- added R2: 10k, Resistor_THT:R_Axial_DIN0207_L6.3mm_D2.5mm_P7.62mm_Horizontal, symbol Device:R_Small_US
- added U3: LCC110, Package_DIP:DIP-8_W7.62mm, symbol Relay_SolidState:LCC110
Connections:
- net GND_BLUE is gone; now on net GND: J1.8, J20.14 (Pin_14)
- net GND_GREEN is gone; now on net GND: J1.7, J20.16 (Pin_16)
- net GND_RED is gone; now on net GND: J1.6, J20.18 (Pin_18)
- net PFW is gone; now on net LPIACT:L1_LP: J20.10 (Pin_10)
- net -10V: now also J2.3 (Pin_3)
- net 5V_TRICKLE: now also D1.2 (A), R2.2, U3.5
- net COMPUTER_5V: now also D2.2 (A); no longer U2.20 (AVCC), U2.7 (VCC)
- net DCO: now also J2.5 (Pin_5)
- net GND: now also H1.1, R1.1, U3.8
- net LINE_SENSE: now also J2.2 (Pin_2)
- net LPIACT:L1_LP: now also J2.6 (Pin_6), U3.6, U3.7
- net PROT: now also J2.4 (Pin_4)
- net at U1.13 (PD7): now also U3.2
- net PWR_BTN: now reaches U1.19 (PB5)
- net PWR_BTN: now also J2.1 (Pin_1), R2.1
- new net: D1.1 (K), D2.1 (K), U2.20 (AVCC), U2.7 (VCC)
- new net: R1.2, U3.3
- no-connect marks 4 -> 40

Commit message: added caps to the board
Parts:
- added C5, C6: 470uF, Capacitor_THT:CP_Radial_D8.0mm_P3.50mm, symbol Device:CP
- added JP1, JP2: SolderJumper_2_Open, Jumper:SolderJumper-2_P1.3mm_Open_RoundedPad1.0x1.5mm, symbol Jumper:SolderJumper_2_Open
Connections:
- net 5V_TRICKLE: now also C5.1
- net COMPUTER_5V: now also C6.1
- net COMPUTER_SCL: now also JP2.2 (B); no longer J1.15
- net COMPUTER_SDA: now also JP1.2 (B); no longer J1.12
- net GND: now also C5.2, C6.2
- new net: J1.12, JP1.1 (A)
- new net: J1.15, JP2.1 (A)
Changed lines of the file:
@@
 	1    0    0    -1
 $EndComp
-Text Label 9500 3800 0    50   ~ 0
+Text Label 9900 3800 0    50   ~ 0
 COMPUTER_SCL
-Text Label 9500 3200 0    50   ~ 0
+Text Label 9900 3200 0    50   ~ 0
 COMPUTER_SDA
 Text Notes 2100 6550 0    50   ~ 0
@@
 GND_RED
 $Comp
-L power:GND #PWR?
+L power:GND #PWR010
 U 1 1 5E77D79F
 P 8350 4950
-F 0 "#PWR?" H 8350 4700 50  0001 C CNN
+F 0 "#PWR010" H 8350 4700 50  0001 C CNN
 F 1 "GND" H 8355 4777 50  0000 C CNN
 F 2 "" H 8350 4950 50  0001 C CNN
@@
 Wire Wire Line
 	8350 4600 8350 4950
+$Comp
+L Device:CP C5
+U 1 1 5E5FB13C
+P 1100 6050
+F 0 "C5" H 1218 6096 50  0000 L CNN
+F 1 "470uF" H 1218 6005 50  0000 L CNN
+F 2 "Capacitor_THT:CP_Radial_D8.0mm_P3.50mm" H 1138 5900 50  0001 C CNN
+F 3 "http://nichicon-us.com/english/products/pdfs/e-upw.pdf" H 1100 6050 50  0001 C CNN
+F 4 "digikey" H 1100 6050 50  0001 C CNN "Vendor"
+F 5 "493-1702-ND" H 1100 6050 50  0001 C CNN "Part#"
+	1    1100 6050
+	1    0    0    -1
+$EndComp
+$Comp
+L Device:CP C6
+U 1 1 5E5FCDDF
+P 1700 6050
+F 0 "C6" H 1818 6096 50  0000 L CNN
+F 1 "470uF" H 1818 6005 50  0000 L CNN
+F 2 "Capacitor_THT:CP_Radial_D8.0mm_P3.50mm" H 1738 5900 50  0001 C CNN
+F 3 "http://nichicon-us.com/english/products/pdfs/e-upw.pdf" H 1700 6050 50  0001 C CNN
+F 4 "digikey" H 1700 6050 50  0001 C CNN "Vendor"
+F 5 "493-1702-ND" H 1700 6050 50  0001 C CNN "Part#"
+	1    1700 6050
+	1    0    0    -1
+$EndComp
+$Comp
+L power:GND #PWR011
+U 1 1 5E5FD400
+P 1450 6550
+F 0 "#PWR011" H 1450 6300 50  0001 C CNN
+F 1 "GND" H 1455 6377 50  0000 C CNN
+F 2 "" H 1450 6550 50  0001 C CNN
+F 3 "" H 1450 6550 50  0001 C CNN
+	1    1450 6550
+	1    0    0    -1
+$EndComp
+Wire Wire Line
+	1700 6200 1700 6550
+Wire Wire Line
+	1700 6550 1450 6550
+Wire Wire Line
+	1100 6200 1100 6550
+Wire Wire Line
+	1100 6550 1450 6550
+Connection ~ 1450 6550
+Text Label 1100 5600 2    50   ~ 0
+5V_TRICKLE
+Text Label 1700 5600 0    50   ~ 0
+COMPUTER_5V
+Wire Wire Line
+	1700 5600 1700 5900
+Wire Wire Line
+	1100 5600 1100 5900
+$Comp
+L Jumper:SolderJumper_2_Open JP1
+U 1 1 5E630257
+P 9650 3200
+F 0 "JP1" H 9650 3405 50  0000 C CNN
+F 1 "SolderJumper_2_Open" H 9650 3314 50  0000 C CNN
+F 2 "Jumper:SolderJumper-2_P1.3mm_Open_RoundedPad1.0x1.5mm" H 9650 3200 50  0001 C CNN
+F 3 "~" H 9650 3200 50  0001 C CNN
+	1    9650 3200
+	1    0    0    -1
+$EndComp
+$Comp
+L Jumper:SolderJumper_2_Open JP2
+U 1 1 5E6323A4
+P 9650 3800
+F 0 "JP2" H 9650 4005 50  0000 C CNN
+F 1 "SolderJumper_2_Open" H 9650 3914 50  0000 C CNN
+F 2 "Jumper:SolderJumper-2_P1.3mm_Open_RoundedPad1.0x1.5mm" H 9650 3800 50  0001 C CNN
+F 3 "~" H 9650 3800 50  0001 C CNN
+	1    9650 3800
+	1    0    0    -1
+$EndComp
+Wire Wire Line
+	9800 3200 9900 3200
+Wire Wire Line
+	9800 3800 9900 3800
 $EndSCHEMATC

Commit message: added J22 board design
Parts:
- J20: Part# 609-2430-ND -> 609-3206-ND
- U3: Part# (none) -> CLA106-ND; part# CLA106-ND -> (none)
Changed lines of the file:
@@
 F 1 "Conn_02x10_Odd_Even" H 8950 2026 50  0000 C CNN
 F 2 "Connector_PinHeader_2.54mm:PinHeader_2x10_P2.54mm_Vertical" H 8900 1500 50  0001 C CNN
-F 3 "https://cdn.amphenol-icc.com/media/wysiwyg/files/drawing/69168.pdf" H 8900 1500 50  0001 C CNN
+F 3 "https://cdn.amphenol-icc.com/media/wysiwyg/files/drawing/67996.pdf" H 8900 1500 50  0001 C CNN
 F 4 "digikey" H 8900 1500 50  0001 C CNN "Vendor"
-F 5 "609-2430-ND" H 8900 1500 50  0001 C CNN "Part#"
+F 5 "609-3206-ND" H 8900 1500 50  0001 C CNN "Part#"
 	1    8900 1500
 	1    0    0    -1
@@
 F 3 "http://www.ixysic.com/home/pdfs.nsf/www/LCC110.pdf/$file/LCC110.pdf" H 2900 4050 50  0001 L CNN
 F 4 "digikey" H 2900 4050 50  0001 C CNN "Vendor"
-F 5 "CLA106-ND" H 2900 4050 50  0001 C CNN "part#"
+F 5 "CLA106-ND" H 2900 4050 50  0001 C CNN "Part#"
 	1    2900 4050
 	1    0    0    -1
