File: schematics_and_pcbs/imac_g3_333mhz_slot_loading_J20_adapter_board/imac_g3_333mhz_slot_loading_J20_adapter_board.sch (KiCad schematic (older format))
At the start: 21 parts, among them J1 Screw_Terminal_01x06, J2 Conn_02x10_Odd_Even, J3 Conn_02x03_Odd_Even, J4 DB15_Female_HighDensity, J5 Conn_02x03_Odd_Even, U1 ATmega328-PU, U2 LCC110, Y1 Crystal

Commit message: updated schematic with a VSYNC detect input line.
Parts:
- added JP3: SolderJumper_2_Open, Jumper:SolderJumper-2_P1.3mm_Open_RoundedPad1.0x1.5mm, symbol Jumper:SolderJumper_2_Open
Connections:
- net V_SYNC: now also JP3.2 (B)
- net at U1.16 (PB2): now also JP3.1 (A)
- no-connect marks 11 -> 10
Other:
- note added: "Sends EDID data to computer via DE15\nconnector and monitors VSYNC to detect\nif computer is on or off."
- note removed: "Sends EDID data to computer via DE15\nconnector"
Changed lines of the file:
@@
 Title "iMac G3 333 Mhz Slot Loading Power and Video Board"
 Date "2020-03-27"
-Rev "2"
+Rev "3"
 Comp ""
 Comment1 "and control other functions."
@@
 COMPUTER_SDA
 Text Notes 3850 6250 0    50   ~ 0
-Sends EDID data to computer via DE15\nconnector
+Sends EDID data to computer via DE15\nconnector and monitors VSYNC to detect\nif computer is on or off.
 NoConn ~ 6550 5700
 Wire Wire Line
@@
 Wire Wire Line
 	4650 1100 4650 1400
-NoConn ~ 4850 2800
 NoConn ~ 4850 3500
 NoConn ~ 4850 3600
@@
 	-1   0    0    1
 $EndComp
+$Comp
+L Jumper:SolderJumper_2_Open JP3
+U 1 1 5E9A08C1
+P 5500 2800
+F 0 "JP3" H 5500 3050 50  0000 C CNN
+F 1 "SolderJumper_2_Open" H 5500 2950 50  0000 C CNN
+F 2 "Jumper:SolderJumper-2_P1.3mm_Open_RoundedPad1.0x1.5mm" H 5500 2800 50  0001 C CNN
+F 3 "~" H 5500 2800 50  0001 C CNN
+	1    5500 2800
+	1    0    0    -1
+$EndComp
+Wire Wire Line
+	5350 2800 4850 2800
+Text Label 5650 2800 0    50   ~ 0
+V_SYNC
 $EndSCHEMATC
