File: schematics_and_pcbs/imac_g3_slot_loading_J22_adapter_board/imac_g3_slot_loading_J22_adapter_board.kicad_pcb (KiCad board)
At the start: 2 copper layers, 65 x 30 mm, 7 parts, among them J1 Conn_02x13_Odd_Even, J2 Screw_Terminal_01x10, J3 AudioJack3, J4 Conn_02x03_Odd_Even

Commit message: fixed miswired microphone jack
Connections:
- J1 pad 1: /-MICROPHONE -> GNDREF
- J3 pad R: /-MICROPHONE -> Net-(J3-PadR)
Routing:
- net /-MICROPHONE: track 11.5 -> 0.00 mm
Other:
- board text added: "Rev 2"
- board text removed: "Rev 1"

Commit message: added electrek mic circuit stuff
Parts:
- added C1: 1uF, Capacitor_THT:CP_Radial_D4.0mm_P1.50mm, F.Cu at (167.8, 90.1)
- added JP1: SolderJumper_2_Open, Jumper:SolderJumper-2_P1.3mm_Open_RoundedPad1.0x1.5mm, B.Cu at (165.0, 95.9)
- added JP2: SolderJumper_3_Open, Jumper:SolderJumper-3_P1.3mm_Open_RoundedPad1.0x1.5mm, B.Cu at (168.3, 102.9)
- added JP3: SolderJumper_2_Open, Jumper:SolderJumper-2_P1.3mm_Open_RoundedPad1.0x1.5mm, B.Cu at (161.3, 99.6)
- added R3: 2.2k, Resistor_THT:R_Axial_DIN0207_L6.3mm_D2.5mm_P7.62mm_Horizontal, F.Cu at (161.3, 95.6)
Connections:
- J3 pad R: Net-(J3-PadR) -> /MICROPHONE_POWER
- J3 pad T: /+MICROPHONE -> Net-(C1-Pad1)
Routing:
- net Net-(C1-Pad1): track 0.00 -> 37.6 mm
- net /+GREEN_LED: track 8.76 -> 45.0 mm, vias 0 -> 2
- net Net-(C1-Pad2): track 0.00 -> 15.0 mm
- net /MICROPHONE_POWER: track 0.00 -> 14.0 mm
- net /+MICROPHONE: track 18.1 -> 22.5 mm
- net Net-(JP1-Pad1): track 0.00 -> 3.20 mm
Other:
- board text added: "1"
- board text added: "1uF"
- board text added: "2"
- board text added: "220"
- board text added: "2k2"
- board text added: "3"

Commit message: updated silkscreen to make it more readable
Other:
- board text added: "PWR BUTTON"
Changed lines of the file:
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@@
   )
   (layers
-    (0 F.Cu signal hide)
+    (0 F.Cu signal)
     (31 B.Cu signal)
     (32 B.Adhes user)
@@
     (effects (font (size 1 1) (thickness 0.15)))
   )
-  (gr_text "GREEN\nLED" (at 120.04 101.64) (layer F.SilkS)
-    (effects (font (size 0.5 0.5) (thickness 0.1)))
-  )
-  (gr_text "POWER\nBUTTON" (at 125.04 101.64) (layer F.SilkS)
-    (effects (font (size 0.5 0.5) (thickness 0.1)))
-  )
-  (gr_text "AMBER\nLED" (at 130.04 101.64) (layer F.SilkS)
-    (effects (font (size 0.5 0.5) (thickness 0.1)))
+  (gr_text "GREEN\nLED" (at 119.84 101.04) (layer F.SilkS)
+    (effects (font (size 0.7 0.7) (thickness 0.15)))
+  )
+  (gr_text "PWR\nBUTTON" (at 125.04 101.64) (layer F.SilkS)
+    (effects (font (size 0.7 0.7) (thickness 0.15)))
+  )
+  (gr_text "AMBER\nLED" (at 130.04 101.24) (layer F.SilkS)
+    (effects (font (size 0.7 0.7) (thickness 0.15)))
   )
   (gr_text GND (at 134.04 101.64) (layer F.SilkS)
@@
     (effects (font (size 1 1) (thickness 0.15)))
   )
-  (gr_text "H2 LEFT" (at 130.022 94.008) (layer F.SilkS)
-    (effects (font (size 0.5 0.5) (thickness 0.1)))
-  )
-  (gr_text "H1 SENSE" (at 130.022 96.548) (layer F.SilkS)
-    (effects (font (size 0.5 0.5) (thickness 0.1)))
-  )
-  (gr_text "H2 RIGHT" (at 119.862 94.008) (layer F.SilkS)
-    (effects (font (size 0.5 0.5) (thickness 0.1)))
-  )
-  (gr_text "H2 SENSE" (at 119.862 96.548) (layer F.SilkS)
-    (effects (font (size 0.5 0.5) (thickness 0.1)))
-  )
-  (gr_text "H1 RIGHT" (at 119.862 99.088) (layer F.SilkS)
-    (effects (font (size 0.5 0.5) (thickness 0.1)))
-  )
-  (gr_text "H1 LEFT" (at 130.022 99.088) (layer F.SilkS)
-    (effects (font (size 0.5 0.5) (thickness 0.1)))
+  (gr_text "H2 LEFT" (at 131.04 94.39) (layer F.SilkS)
+    (effects (font (size 1 1) (thickness 0.15)))
+  )
+  (gr_text "H1 SENSE" (at 131.79 96.548) (layer F.SilkS)
+    (effects (font (size 1 1) (thickness 0.15)))
+  )
+  (gr_text "H2 RIGHT" (at 118.29 93.89) (layer F.SilkS)
+    (effects (font (size 1 1) (thickness 0.15)))
+  )
+  (gr_text "H2 SENSE" (at 118.04 96.548) (layer F.SilkS)
+    (effects (font (size 1 1) (thickness 0.15)))
+  )
+  (gr_text "H1 RIGHT" (at 118.44 99.04) (layer F.SilkS)
+    (effects (font (size 1 1) (thickness 0.15)))
+  )
+  (gr_text "H1 LEFT" (at 131.24 99.04) (layer F.SilkS)
+    (effects (font (size 1 1) (thickness 0.15)))
   )
   (gr_line (start 112.242 114.328) (end 105.892 114.328) (layer F.SilkS) (width 0.12))
